File: Hardware/MicroMod_Sno_Processor.sch (EAGLE design)
At the start: 35 parts, among them IC1 FT230XQ, J1 MICROMOD-2222, J2 CORTEX_JTAG_DEBUG_PTH_NS, Q1 RE1C001ZP, U2 OSC_TINY_16

Commit message: V10 Update
Updated routing for DFM and proto issues
Parts:
- added LOGO2: SFE_LOGO_FLAME.1_INCH, SparkFun-Aesthetics:SFE_LOGO_FLAME.1_INCH
- Q1: value RE1C001ZP -> 20V/0.1A
- R10: value 22 -> 22OHM-0402T-1/16W-1%; device New_Parts:22OHM-0402_TIGHT-1/10W-1% -> SparkFun-Resistors:22OHM-0402T-1/16W-1%
- U2: value OSC_TINY_16 -> 16MHz
Connections:
- net LED renamed STAT
- removed net TXLED: IC1.CBUS2
Other:
- note added: "Alorium Technology"
- note added: "FPGA Power"
- note added: "V10"
- note removed: "3.3 Volt"
- note removed: "FPGA Power & GND"
- note removed: "V In"
- moved on the sheet: C10, C11, C12, C2, C3, C4, C6, C7, C8, C9, IC1, J1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

Commit message: V10 QC changes
- Added voltage range to FPGA
- Updated RX LED to yellow
- Updated PROD_ID for 22 ohm resistor
Parts:
- R10: value 22OHM-0402T-1/16W-1% -> 22
- RX: value BLUE -> Yellow; device SparkFun-LED:LED-BLUE0603 -> SparkFun-LED:LED-YELLOW0603
Other:
- note added: "VCC: 2.85 - 3.465V"
Changed lines of the file:
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@@
 <?xml version="1.0" encoding="utf-8"?>
 <!DOCTYPE eagle SYSTEM "eagle.dtd">
-<eagle version="9.6.2">
+<eagle version="9.5.2">
 <drawing>
 <settings>
@@
 <part name="GND5" library="SparkFun-PowerSymbols" deviceset="GND" device=""/>
 <part name="R9" library="SparkFun-Resistors" deviceset="1KOHM" device="-0402T-1/16W-1%" value="1k"/>
-<part name="R10" library="SparkFun-Resistors" deviceset="22OHM" device="-0402T-1/16W-1%" value="22OHM-0402T-1/16W-1%"/>
+<part name="R10" library="SparkFun-Resistors" deviceset="22OHM" device="-0402T-1/16W-1%" value="22"/>
 <part name="C8" library="SparkFun-Capacitors" deviceset="0.5PF" device="-0402_TIGHT-50V-PM0.05PF-NP0" value="0.5pF"/>
 <part name="GND10" library="SparkFun-PowerSymbols" deviceset="GND" device=""/>
@@
 <part name="Q1" library="New_Parts" deviceset="RE1C001ZP" device="" value="20V/0.1A"/>
 <part name="R1" library="SparkFun-Resistors" deviceset="1KOHM" device="-0402T-1/16W-1%" value="1k"/>
-<part name="RX" library="SparkFun-LED" deviceset="LED-BLUE" device="0603" value="BLUE"/>
+<part name="RX" library="SparkFun-LED" deviceset="LED-YELLOW" device="0603" value="Yellow"/>
 <part name="FID1" library="SparkFun-Aesthetics" deviceset="FIDUCIAL" device="1X2"/>
 <part name="FID2" library="SparkFun-Aesthetics" deviceset="FIDUCIAL" device="1X2"/>
@@
 <wire x1="330.2" y1="187.96" x2="330.2" y2="279.4" width="0.2032" layer="97" style="longdash"/>
 <text x="353.568" y="11.43" size="2.54" layer="94" font="vector">Alorium Technology</text>
+<text x="96.52" y="76.2" size="2.54" layer="97">VCC: 2.85 - 3.465V</text>
 </plain>
 <instances>
@@
 <instance part="R10" gate="G$1" x="195.58" y="25.4" smashed="yes">
 <attribute name="NAME" x="195.58" y="26.924" size="1.778" layer="95" font="vector" align="bottom-center"/>
+<attribute name="VALUE" x="195.58" y="23.876" size="1.778" layer="96" font="vector" align="top-center"/>
 </instance>
 <instance part="C8" gate="G$1" x="205.74" y="17.78" smashed="yes" rot="MR0">

Commit message: Updated oscillator
Updated oscillator to a smaller 2.0x1.6mm package
Parts:
- U2: device New_Parts:OSC_TINY_16 -> New_Parts:OSC_TINY_16SMD20X16
Other:
- note removed: "VCC: 2.85 - 3.465V"
Changed lines of the file:
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@@
 <part name="C12" library="SparkFun-Capacitors" deviceset="0.1UF" device="-0402T-6.3V-10%-X7R" value="0.1uF"/>
 <part name="J1" library="SparkFun-MicroMod" deviceset="MICROMOD" device="-2222"/>
-<part name="U2" library="New_Parts" deviceset="OSC_TINY_16" device="" value="16MHz"/>
+<part name="U2" library="New_Parts" deviceset="OSC_TINY_16" device="SMD20X16" value="16MHz"/>
 <part name="IC1" library="New_Parts" deviceset="FT230X" device="Q" package3d_urn="urn:adsk.eagle:package:14017/1" value="FT230XQ"/>
 <part name="GND2" library="SparkFun-PowerSymbols" deviceset="GND" device=""/>
@@
 <wire x1="330.2" y1="187.96" x2="330.2" y2="279.4" width="0.2032" layer="97" style="longdash"/>
 <text x="353.568" y="11.43" size="2.54" layer="94" font="vector">Alorium Technology</text>
-<text x="96.52" y="76.2" size="2.54" layer="97">VCC: 2.85 - 3.465V</text>
 </plain>
 <instances>

Commit message: Update MicroMod_Sno_Processor.sch
Added VCC range note back to schematic
Other:
- note added: "VCC: 2.85 - 3.465V"
Changed lines of the file:
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@@
 <wire x1="330.2" y1="187.96" x2="330.2" y2="279.4" width="0.2032" layer="97" style="longdash"/>
 <text x="353.568" y="11.43" size="2.54" layer="94" font="vector">Alorium Technology</text>
+<text x="96.52" y="76.2" size="2.54" layer="97" font="vector">VCC: 2.85 - 3.465V</text>
 </plain>
 <instances>
